File: Kicad_Eduino_FPGA.kicad_pcb (KiCad board)
At the start: 4 copper layers, 99 x 49 mm, 177 parts, among them J1 Conn_02x05_Odd_Even, J10 Conn_02x05_Odd_Even, J12 Conn_01x06, J13 Barrel_Jack_Switch, J2 Conn_02x05_Odd_Even, J3 Conn_02x05_Odd_Even, J4 USB_C_Receptacle_USB2.0, J5 Conn_02x05_Odd_Even, J7 Conn_02x05_Odd_Even, J8 Conn_02x05_Odd_Even, J9 Conn_02x05_Odd_Even, Q1 Q_DUAL_PNP_PNP_C1B1B2C2E2E1, Q2 DMG2305UXQ-7, Q3 DTC143Z, U1 XC6SLX4-TQG144, U10 Nexperia 74LVC1G126GV,125, U11 SN74AHC1G04DBVR, U12 74LVC1G157_1, U13 LMC555CMMX/NOPB, U14 SN74AHC1G04DBVR, U15 SN74AHC1G04DBVR, U16 SN74AHC1G04DBVR, U2 W25Q128JVSIQ, U3 LY68L6400 (64MBits QSPI), U4 AZ1117-1.2, U5 AZ1117-3.3, U6 AZ1117-3.3, U7 TPS54302DDCR, U8 74HC244, U9 CH340G, X1 50MHz 3225 4P Oscillator, Y1 12MHz

Commit message: updating to repo for Bob# Please enter the commit message for your changes. Lines starting# with '#' will be ignored, and an empty message aborts the commit.## On branch main# Your branch is up to date with 'origin/main'.## Changes to be committed:#	modified:   Kicad_Eduino_FPGA.csv#	modified:   Kicad_Eduino_FPGA.kicad_pcb#	modified:   Kicad_Eduino_FPGA.kicad_prl#	modified:   Kicad_Eduino_FPGA.kicad_pro#	modified:   Kicad_Eduino_FPGA.kicad_sch## Changes not staged for commit:#	deleted:    Kicad_Eduino_FPGA-backups/Kicad_Eduino_FPGA-2021-02-09_232526.zip#	deleted:    Kicad_Eduino_FPGA-backups/Kicad_Eduino_FPGA-2021-02-09_233339.zip#	deleted:    Kicad_Eduino_FPGA-backups/Kicad_Eduino_FPGA-2021-02-09_234305.zip#	deleted:    Kicad_Eduino_FPGA-backups/Kicad_Eduino_FPGA-2021-02-09_234829.zip#	deleted:    Kicad_Eduino_FPGA-backups/Kicad_Eduino_FPGA-2021-02-10_225322.zip#	deleted:    Kicad_Eduino_FPGA-backups/Kicad_Eduino_FPGA-2021-02-10_230338.zip#	deleted:    Kicad_Eduino_FPGA-backups/Kicad_Eduino_FPGA-2021-02-10_231635.zip#	deleted:    Kicad_Eduino_FPGA-backups/Kicad_Eduino_FPGA-2021-02-10_235033.zip#	deleted:    Kicad_Eduino_FPGA-backups/Kicad_Eduino_FPGA-2021-02-10_235700.zip#	deleted:    Kicad_Eduino_FPGA-backups/Kicad_Eduino_FPGA-2021-02-11_194504.zip#	deleted:    Kicad_Eduino_FPGA-backups/Kicad_Eduino_FPGA-2021-02-11_195144.zip#	deleted:    Kicad_Eduino_FPGA-backups/Kicad_Eduino_FPGA-2021-02-11_195810.zip#	deleted:    Kicad_Eduino_FPGA-backups/Kicad_Eduino_FPGA-2021-02-11_200450.zip#	deleted:    Kicad_Eduino_FPGA-backups/Kicad_Eduino_FPGA-2021-02-11_212659.zip#	deleted:    Kicad_Eduino_FPGA-backups/Kicad_Eduino_FPGA-2021-02-12_233121.zip#	deleted:    Kicad_Eduino_FPGA-backups/Kicad_Eduino_FPGA-2021-02-12_233747.zip#	deleted:    Kicad_Eduino_FPGA-backups/Kicad_Eduino_FPGA-2021-02-12_234412.zip#	deleted:    Kicad_Eduino_FPGA-backups/Kicad_Eduino_FPGA-2021-02-12_235106.zip#	deleted:    Kicad_Eduino_FPGA-backups/Kicad_Eduino_FPGA-2021-02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
Parts:
- removed J13: Barrel_Jack_Switch, Connector_BarrelJack:BarrelJack_Horizontal
- added C46: 1n0/50V, Capacitor_SMD:C_0603_1608Metric, F.Cu at (85.6, 177.6)
- added J6: Barrel_Jack_Switch, Connector_BarrelJack:BarrelJack_Horizontal, F.Cu at (145.9, 161.3)
- added R66: 100R, Resistor_SMD:R_0603_1608Metric, F.Cu at (134.4, 175.0)
- added R67: 100R, Resistor_SMD:R_0603_1608Metric, F.Cu at (134.4, 173.4)
- added R68: 0R, Resistor_SMD:R_0603_1608Metric, F.Cu at (92.2, 169.2)
- C43, C44: value 2n2/50V -> 1n0/50V
- D16: value D_Small -> SS14
- R54: value 0R -> 1K0
- X1: value 50MHz 3225 4P Oscillator -> 20MHz 3225 4P Oscillator
- moved C3 60.7 mm to (124.2, 160.2)
- moved C1 39.0 mm to (128.6, 147.2), turned to 90 degrees
- moved R20 3.79 mm to (126.4, 175.8), turned to -90 degrees
- moved R54 2.38 mm to (87.8, 176.8), turned to -90 degrees
- moved C28 1.90 mm to (92.6, 165.6)
- moved C4 1.88 mm to (90.9, 165.6)
- moved R55 0.60 mm to (89.8, 170.0)
Connections:
- net DCD renamed DONE_2
- net DTR renamed PROGRAM_B_2
- net JTAG_GND renamed GND
- net VINT_REGOUT renamed Net-(C12-Pad1)
- net Vdrive_regout renamed Net-(C13-Pad1)
- C10 pad 1: JTAG_VAUX -> 3V3
- C11 pad 1: JTAG_VAUX -> 3V3
- C26 pad 1: JTAG_VAUX -> 3V3
- C45 pad 1: JTAG_VAUX -> 3V3
- C9 pad 1: JTAG_VAUX -> 3V3
- R19 pad 2: FPGA_CLOCK -> USER_CLOCK
- R2 pad 1: FPGA_CLOCK -> USER_CLOCK
- R20 pad 1: FPGA_CLOCK -> USER_CLOCK
- R25 pad 1: 3V3 -> JTAG_VAUX
- R3 pad 1: JTAG_VAUX -> 3V3
- R4 pad 1: JTAG_VAUX -> 3V3
- R5 pad 1: JTAG_VAUX -> 3V3
- R53 pad 1: JTAG_VAUX -> 3V3
- R54 pad 1: TRIG_555 -> 3V3
- R65 pad 2: JTAG_VAUX -> 3V3
- U1 pad 55: FPGA_CLOCK -> USER_CLOCK
- U1 pad 66: unconnected-(U1-Pad66) -> RX
- U10 pad 1: unconnected-(U10-Pad1) -> Net-(R68-Pad2)
- U10 pad 5: JTAG_VAUX -> 3V3
- U11 pad 5: JTAG_VAUX -> 3V3
- U12 pad 5: JTAG_VAUX -> 3V3
- U13 pad 4: JTAG_VAUX -> 3V3
- U13 pad 8: JTAG_VAUX -> 3V3
- U14 pad 5: JTAG_VAUX -> 3V3
- U15 pad 5: JTAG_VAUX -> 3V3
- U16 pad 5: JTAG_VAUX -> 3V3
- U2 pad 6: FPGA_CLOCK -> FPGA_CCLK
- U2 pad 8: JTAG_VAUX -> 3V3
- U9 pad 11: RI -> INIT_B_2
- U9 pad 16: JTAG_VAUX -> 3V3
- U9 pad 4: JTAG_VAUX -> 3V3
- X1 pad 1: JTAG_VAUX -> 3V3
- X1 pad 4: JTAG_VAUX -> 3V3
Routing:
- net JTAG_VAUX: track 424.0 -> 213.2 mm, vias 15 -> 9
- net 3V3: track 136.6 -> 206.8 mm, vias 24 -> 38
- net RX: track 0.00 -> 50.6 mm, vias 0 -> 2
- net INIT_B_2: track 2.93 -> 49.7 mm, vias 0 -> 2
- net FPGA_CLOCK: track 46.5 -> 0.00 mm, vias 2 -> 0
- net 5V0: track 272.3 -> 229.3 mm
- net USER_CLOCK: track 0.00 -> 26.9 mm, vias 0 -> 2
- net FPGA_CCLK: track 28.9 -> 53.8 mm
- net FPGA_M1: track 26.5 -> 48.5 mm, vias 2 -> 3
- net Net-(C12-Pad1): track 60.9 -> 39.7 mm, vias 5 -> 3
- net GND: track 381.8 -> 364.2 mm, vias 88 -> 105
- net PROGRAM_B_2: track 67.2 -> 52.8 mm
- net Net-(R68-Pad2): track 0.00 -> 5.65 mm
- net VINT_1V2: track 142.8 -> 147.4 mm, vias 9 -> 10
- net SPIRAM_SCK: track 32.5 -> 28.4 mm
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