File: Kicad_Eduino_FPGA.kicad_sch (KiCad schematic)
At the start: 31 parts, among them U1 XC6SLX4-TQG144, U2 W25Q128JVSIQ, U3 LY68L6400 (64MBits QSPI), X1 50MHz 3225 4P Oscillator

Commit message: updating to repo for Bob# Please enter the commit message for your changes. Lines starting# with '#' will be ignored, and an empty message aborts the commit.## On branch main# Your branch is up to date with 'origin/main'.## Changes to be committed:#	modified:   Kicad_Eduino_FPGA.csv#	modified:   Kicad_Eduino_FPGA.kicad_pcb#	modified:   Kicad_Eduino_FPGA.kicad_prl#	modified:   Kicad_Eduino_FPGA.kicad_pro#	modified:   Kicad_Eduino_FPGA.kicad_sch## Changes not staged for commit:#	deleted:    Kicad_Eduino_FPGA-backups/Kicad_Eduino_FPGA-2021-02-09_232526.zip#	deleted:    Kicad_Eduino_FPGA-backups/Kicad_Eduino_FPGA-2021-02-09_233339.zip#	deleted:    Kicad_Eduino_FPGA-backups/Kicad_Eduino_FPGA-2021-02-09_234305.zip#	deleted:    Kicad_Eduino_FPGA-backups/Kicad_Eduino_FPGA-2021-02-09_234829.zip#	deleted:    Kicad_Eduino_FPGA-backups/Kicad_Eduino_FPGA-2021-02-10_225322.zip#	deleted:    Kicad_Eduino_FPGA-backups/Kicad_Eduino_FPGA-2021-02-10_230338.zip#	deleted:    Kicad_Eduino_FPGA-backups/Kicad_Eduino_FPGA-2021-02-10_231635.zip#	deleted:    Kicad_Eduino_FPGA-backups/Kicad_Eduino_FPGA-2021-02-10_235033.zip#	deleted:    Kicad_Eduino_FPGA-backups/Kicad_Eduino_FPGA-2021-02-10_235700.zip#	deleted:    Kicad_Eduino_FPGA-backups/Kicad_Eduino_FPGA-2021-02-11_194504.zip#	deleted:    Kicad_Eduino_FPGA-backups/Kicad_Eduino_FPGA-2021-02-11_195144.zip#	deleted:    Kicad_Eduino_FPGA-backups/Kicad_Eduino_FPGA-2021-02-11_195810.zip#	deleted:    Kicad_Eduino_FPGA-backups/Kicad_Eduino_FPGA-2021-02-11_200450.zip#	deleted:    Kicad_Eduino_FPGA-backups/Kicad_Eduino_FPGA-2021-02-11_212659.zip#	deleted:    Kicad_Eduino_FPGA-backups/Kicad_Eduino_FPGA-2021-02-12_233121.zip#	deleted:    Kicad_Eduino_FPGA-backups/Kicad_Eduino_FPGA-2021-02-12_233747.zip#	deleted:    Kicad_Eduino_FPGA-backups/Kicad_Eduino_FPGA-2021-02-12_234412.zip#	deleted:    Kicad_Eduino_FPGA-backups/Kicad_Eduino_FPGA-2021-02-12_235106.zip#	deleted:    Kicad_Eduino_FPGA-backups/Kicad_Eduino_FPGA-2021-02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
Parts:
- removed C10, C11: 1uF/50V, Capacitor_SMD:C_0603_1608Metric, symbol Device:C_Small
- removed R3, R4, R5: 4k7, Resistor_SMD:R_0603_1608Metric, symbol Device:R_Small
- removed U2: W25Q128JVSIQ, Package_SO:SOIC-8_5.275x5.275mm_P1.27mm, symbol Memory_Flash:W25Q128JVS
- added H1, H2, H3, H4: MountingHole_Pad, MountingHole:MountingHole_3mm_Pad_Via, symbol Mechanical:MountingHole_Pad
- added J1, J10, J2, J3, J5, J7, J8, J9: Conn_02x05_Odd_Even, MAKER40X40_PCB_SYSTEM:PinHeader_2x05_P2.00mm_Vertical_edwin, symbol Connector_Generic:Conn_02x05_Odd_Even
- added J12: Conn_01x06, Connector_PinHeader_2.54mm:PinHeader_1x06_P2.54mm_Vertical, symbol Connector_Generic:Conn_01x06
- added R57, R58: 0R, Resistor_SMD:R_0603_1608Metric, symbol Device:R_Small
- added RN1, RN2, RN3, RN6, RN8, RN9: 33R, Resistor_SMD:R_Array_Concave_4x0402, symbol Device:R_Pack04
- added TP1, TP2, TP3, TP4, TP5, TP6, TP7, TP8: TestPoint, TestPoint:TestPoint_Pad_2.0x2.0mm, symbol Connector:TestPoint
- added U15, U16: SN74AHC1G04DBVR, Package_TO_SOT_SMD:SOT-23-5, symbol 74xGxx:SN74LVC1G14DBV
- X1: value 50MHz 3225 4P Oscillator -> 20MHz 3225 4P Oscillator; LCSC C26431 -> C32529; MFG_PART SIT1602AI-22-33E-50.000000D -> Q33310F70051500
Connections:
- net +3V3: now also R25.1, J12.6 (Pin_6); no longer C9.1, R65.2, X1.1 (~ST), X1.4 (VCC)
- net GND: now also H1.1, J1.1 (Pin_1), J1.10 (Pin_10), J10.1 (Pin_1), J10.10 (Pin_10), J12.5 (Pin_5), J2.1 (Pin_1), J2.10 (Pin_10), J3.1 (Pin_1), J3.10 (Pin_10), J5.1 (Pin_1), J5.10 (Pin_10), J7.1 (Pin_1), J7.10 (Pin_10), J8.1 (Pin_1), J8.10 (Pin_10), J9.1 (Pin_1), J9.10 (Pin_10), U15.3 (GND), U16.3 (GND)
- net JTAG_TCK: now also J12.4 (Pin_4)
- net JTAG_TDI: now also J12.2 (Pin_2)
- net JTAG_TDO: now also J12.3 (Pin_3)
- net JTAG_TMS: now also J12.1 (Pin_1)
- net L32N: now also RN8.7 (R2.2)
- net L32P: now also RN8.8 (R1.2)
- net L33N: now also RN8.5 (R4.2)
- net L33P: now also RN8.6 (R3.2)
- net L34N: now also RN9.7 (R2.2)
- net L34P: now also RN9.8 (R1.2)
- net L40N: now also RN9.5 (R4.2)
- net L40P: now also RN9.6 (R3.2)
- net L41N: now also RN1.7 (R2.2)
- net L41P: now also RN1.8 (R1.2)
- net L42N: now also RN1.5 (R4.2)
- net L42P: now also RN1.6 (R3.2)
- net L43N: now also RN2.7 (R2.2)
- net L43P: now also RN2.8 (R1.2)
- net L45N: now also RN2.5 (R4.2)
- net L45P: now also RN2.6 (R3.2)
- net L48N: now also J5.4 (Pin_4)
- net L48P: now also J5.2 (Pin_2)
- net L49N: now also J5.8 (Pin_8)
- net L49P: now also J5.6 (Pin_6)
- net L50N: now also RN3.7 (R2.2)
- net L50P: now also RN3.8 (R1.2)
- net L51N: now also RN3.5 (R4.2)
- net L51P: now also RN3.6 (R3.2)
- net L52N: now also RN6.2 (R2.1)
- net L52P: now also RN6.1 (R1.1)
- net L62N: now also J8.4 (Pin_4)
- net L62P: now also J8.2 (Pin_2)
- net L64N: now also J8.8 (Pin_8)
- net L64P: now also J8.6 (Pin_6)
- net L83N: now also RN6.4 (R4.1)
- net L83P: now also RN6.3 (R3.1)
- net Vdrive: now also C9.1, R65.2, X1.1 (~ST), X1.4 (VCC), U15.5 (VCC), U16.5 (VCC); no longer R25.1
- net RX: now reaches U1.66 (IO_L2N_CMPMOSI_2)
- net DCD renamed DONE_2
- net DTR renamed PROGRAM_B_2
- net FPGA_CLOCK renamed USER_CLOCK
- new net: J1.2 (Pin_2), RN1.1 (R1.1)
- new net: J1.4 (Pin_4), RN1.2 (R2.1)
- new net: J1.6 (Pin_6), RN1.3 (R3.1)
- new net: J1.8 (Pin_8), RN1.4 (R4.1)
- new net: J2.2 (Pin_2), RN2.1 (R1.1)
- new net: J2.4 (Pin_4), RN2.2 (R2.1)
- new net: J2.6 (Pin_6), RN2.3 (R3.1)
- new net: J2.8 (Pin_8), RN2.4 (R4.1)
- new net: J7.2 (Pin_2), RN6.8 (R1.2)
- new net: J7.4 (Pin_4), RN6.7 (R2.2)
- new net: J7.6 (Pin_6), RN6.6 (R3.2)
- new net: J7.8 (Pin_8), RN6.5 (R4.2)
- new net: R57.1, TP3.1
- new net: R57.2, TP4.1
- new net: J3.2 (Pin_2), RN3.1 (R1.1)
- new net: J3.4 (Pin_4), RN3.2 (R2.1)
- new net: J3.6 (Pin_6), RN3.3 (R3.1)
- new net: J3.8 (Pin_8), RN3.4 (R4.1)
- new net: TP1.1, U15.2
- new net: TP2.1, U15.4
- new net: TP8.1, U16.4
- new net: J10.2 (Pin_2), RN9.1 (R1.1)
- new net: J10.4 (Pin_4), RN9.2 (R2.1)
- new net: J10.6 (Pin_6), RN9.3 (R3.1)
- new net: J10.8 (Pin_8), RN9.4 (R4.1)
- new net: J9.2 (Pin_2), RN8.1 (R1.1)
- new net: J9.4 (Pin_4), RN8.2 (R2.1)
- new net: J9.6 (Pin_6), RN8.3 (R3.1)
- new net: J9.8 (Pin_8), RN8.4 (R4.1)
- new net: R58.1, TP6.1
- new net: R58.2, TP7.1
- new net: TP5.1, U16.2
- new net 3V3: J1.3 (Pin_3), J1.5 (Pin_5), J10.3 (Pin_3), J10.5 (Pin_5), J2.3 (Pin_3), J2.5 (Pin_5), J3.3 (Pin_3), J3.5 (Pin_5), J5.3 (Pin_3), J5.5 (Pin_5), J7.3 (Pin_3), J7.5 (Pin_5), J8.3 (Pin_3), J8.5 (Pin_5), J9.3 (Pin_3), J9.5 (Pin_5)
- new net 5V0: J1.7 (Pin_7), J1.9 (Pin_9), J10.7 (Pin_7), J10.9 (Pin_9), J2.7 (Pin_7), J2.9 (Pin_9), J3.7 (Pin_7), J3.9 (Pin_9), J5.7 (Pin_7), J5.9 (Pin_9), J7.7 (Pin_7), J7.9 (Pin_9), J8.7 (Pin_7), J8.9 (Pin_9), J9.7 (Pin_7), J9.9 (Pin_9)
- no-connect marks 0 -> 53
Other:
- removed sheet Mounting_holes
- removed sheet SheetConnectors
- removed sheet SheetPower
- added sheet LogicalLedsFPGA (Eduino_LEDS_fpga.kicad_sch)
- added sheet PowerBusLeds (Eduino_PwrBusLeds.kicad_sch)
- added sheet PowerSupply (Eduino_PSU.kicad_sch)
- added sheet Serial_USB (Serial_USB_magic.kicad_sch)
- note added: "Bread-Board Area"
- note added: "JTAG for access to FPGA"
- note added: "LEFT / BOTTOM Connected to Ground Other holes insulated"
- note removed: "BOOT_FLASH"
- moved on the sheet: C9, D9, R19, R2, R20, R25, R26, R27, R28, R39, R40, R41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
